Commit message: URDF modified

File: mower.urdf (robot description, URDF)
Before this commit: robot autonomous_lawnmower, 6 links, 5 joints
Links:
- removed link front_camera
- added link front_bottom_camera, mass 0.1; collision box size=0.05 0.05 0.05; visual box size=0.05 0.05 0.05
- added link rear_bottom_camera, mass 0.1; collision box size=0.05 0.05 0.05; visual box size=0.05 0.05 0.05
Joints:
- removed joint front_camera_joint
- added joint front_bottom_camera_joint: type fixed, parent base_link, child front_bottom_camera, origin xyz=0.4 -0 -0.01 rpy=0 0 0
- added joint rear_bottom_camera_joint: type fixed, parent base_link, child rear_bottom_camera, origin xyz=-0.4 0 -0.01 rpy=0 0 0
- joint front_left_wheel_joint: origin xyz=-0.4 0.45 0 rpy=0 0 0 -> xyz=-0.4 0.45 -0.05 rpy=0 0 0
- joint front_right_wheel_joint: origin xyz=-0.4 -0.45 0 rpy=0 0 0 -> xyz=-0.4 -0.45 -0.05 rpy=0 0 0
- joint left_drive_wheel_joint: origin xyz=0.4 0.45 0 rpy=0 0 0 -> xyz=0.4 0.45 -0.05 rpy=0 0 0
- joint right_drive_wheel_joint: origin xyz=0.4 -0.45 0 rpy=0 0 0 -> xyz=0.4 -0.45 -0.05 rpy=0 0 0

Commit message: URDF changed

File: mower.urdf (robot description, URDF)
Before this commit: robot autonomous_lawnmower, 7 links, 6 joints
Links:
- link front_left_wheel: geometry collision cylinder length=0.1 radius=0.3; visual cylinder length=0.1 radius=0.3
- link front_right_wheel: geometry collision cylinder length=0.1 radius=0.3; visual cylinder length=0.1 radius=0.3
- link left_drive_wheel: geometry collision cylinder length=0.1 radius=0.3; visual cylinder length=0.1 radius=0.3
- link right_drive_wheel: geometry collision cylinder length=0.1 radius=0.3; visual cylinder length=0.1 radius=0.3
Joints:
- joint front_bottom_camera_joint: origin xyz=0.4 -0 -0.01 rpy=0 0 0 -> xyz=0.4 -0 -0.025 rpy=0 0 0
- joint rear_bottom_camera_joint: origin xyz=-0.4 0 -0.01 rpy=0 0 0 -> xyz=-0.4 0 -0.025 rpy=0 0 0

Commit message: URDF changed

File: mower.urdf (robot description, URDF)
Before this commit: robot autonomous_lawnmower, 7 links, 6 joints
Joints:
- joint front_bottom_camera_joint: origin xyz=0.4 -0 -0.025 rpy=0 0 0 -> xyz=0.4 0 -0.025 rpy=1.5708 0 0
- joint rear_bottom_camera_joint: origin xyz=-0.4 0 -0.025 rpy=0 0 0 -> xyz=-0.4 0 -0.025 rpy=1.5708 0 0

Commit message: URDF changed

File: mower.urdf (robot description, URDF)
Before this commit: robot autonomous_lawnmower, 7 links, 6 joints
Joints:
- joint front_bottom_camera_joint: origin xyz=0.4 0 -0.025 rpy=1.5708 0 0 -> xyz=0.4 0 -0.025 rpy=0 1.5708 0
- joint rear_bottom_camera_joint: origin xyz=-0.4 0 -0.025 rpy=1.5708 0 0 -> xyz=-0.4 0 -0.025 rpy=0 1.5708 0
